File: matrix.sch (KiCad schematic (older format))
At the start: 130 parts, among them K1 ESC, K10 #9, K11 #0, K12 MINUS, K13 PLUS, K14 TAB, K15 Q, K16 W, K17 E, K18 R, K19 T, K2 #1, K20 Y, K21 U, K22 I, K23 O, K24 P, K25 [, K26 ], K27 CAPS, K28 A, K29 S, K3 #2, K30 D, K31 F, K32 G, K33 H, K34 J, K35 K, K36 L, K37 SEMICOLON, K38 QUOTE, K39 ENTER, K4 #3, K40 LSHIFT, K41 Z, K42 X, K43 C, K44 V, K45 B, K46 N, K47 M, K48 COMMA, K49 DOT, K5 #4, K50 SLASH, K51 RSHIFT, K52 BACKSLASH, K53 LCTL, K54 LGUI, K55 LALT, K56 FN2, K57 LSPC, K58 RSPC, K59 RALT, K6 #5, K60 RGUI, K61 LEFT, K62 DOWN, K63 RIGHT, K64 UP, K65 BKSPC, K7 #6, K8 #7, K9 #8

Commit message: Update labels on footprints
Parts:
- K14, K51, K52, K53, K54, K55: footprint xeal_components:MX-Choc-1U -> xeal_components:MX-Choc-1.5U
- K27: footprint xeal_components:MX-Choc-1U -> xeal_components:MX-Alps-Choc-2U-pin-flip
- K40: footprint xeal_components:MX-Alps-Choc-2U-pin-flip -> xeal_components:MX-Choc-2.5U-pin21
- K56: footprint xeal_components:MX-Choc-1U -> xeal_components:MX-Alps-Choc-2U-stabflip-pinflip
- K57, K58: footprint xeal_components:MX-Alps-Choc-2U-no-led -> xeal_components:MX-Alps-Choc-2U-stabflip-pinflip
Changed lines of the file:
@@
 F 0 "K14" H 2050 2900 50  0000 C CNN
 F 1 "TAB" H 2050 2794 50  0000 C CNN
-F 2 "xeal_components:MX-Choc-1U" H 2050 2650 50  0001 C CNN
+F 2 "xeal_components:MX-Choc-1.5U" H 2050 2650 50  0001 C CNN
 F 3 "~" H 2050 2650 50  0001 C CNN
 	1    2050 2650
@@
 F 0 "K27" H 2050 3650 50  0000 C CNN
 F 1 "CAPS" H 2050 3544 50  0000 C CNN
-F 2 "xeal_components:MX-Choc-1U" H 2050 3400 50  0001 C CNN
+F 2 "xeal_components:MX-Alps-Choc-2U-pin-flip" H 2050 3400 50  0001 C CNN
 F 3 "~" H 2050 3400 50  0001 C CNN
 	1    2050 3400
@@
 F 0 "K40" H 2050 4400 50  0000 C CNN
 F 1 "LSHIFT" H 2050 4294 50  0000 C CNN
-F 2 "xeal_components:MX-Alps-Choc-2U-pin-flip" H 2050 4150 50  0001 C CNN
+F 2 "xeal_components:MX-Choc-2.5U-pin21" H 2050 4150 50  0001 C CNN
 F 3 "~" H 2050 4150 50  0001 C CNN
 	1    2050 4150
@@
 F 0 "K51" H 7550 4400 50  0000 C CNN
 F 1 "RSHIFT" H 7550 4294 50  0000 C CNN
-F 2 "xeal_components:MX-Choc-1U" H 7550 4150 50  0001 C CNN
+F 2 "xeal_components:MX-Choc-1.5U" H 7550 4150 50  0001 C CNN
 F 3 "~" H 7550 4150 50  0001 C CNN
 	1    7550 4150
@@
 F 0 "K52" H 8050 4400 50  0000 C CNN
 F 1 "BACKSLASH" H 8050 4294 50  0000 C CNN
-F 2 "xeal_components:MX-Choc-1U" H 8050 4150 50  0001 C CNN
+F 2 "xeal_components:MX-Choc-1.5U" H 8050 4150 50  0001 C CNN
 F 3 "~" H 8050 4150 50  0001 C CNN
 	1    8050 4150
@@
 F 0 "K53" H 2050 5150 50  0000 C CNN
 F 1 "LCTL" H 2050 5044 50  0000 C CNN
-F 2 "xeal_components:MX-Choc-1U" H 2050 4900 50  0001 C CNN
+F 2 "xeal_components:MX-Choc-1.5U" H 2050 4900 50  0001 C CNN
 F 3 "~" H 2050 4900 50  0001 C CNN
 	1    2050 4900
@@
 F 0 "K54" H 2550 5150 50  0000 C CNN
 F 1 "LGUI" H 2550 5044 50  0000 C CNN
-F 2 "xeal_components:MX-Choc-1U" H 2550 4900 50  0001 C CNN
+F 2 "xeal_components:MX-Choc-1.5U" H 2550 4900 50  0001 C CNN
 F 3 "~" H 2550 4900 50  0001 C CNN
 	1    2550 4900
@@
 F 0 "K55" H 3050 5150 50  0000 C CNN
 F 1 "LALT" H 3050 5044 50  0000 C CNN
-F 2 "xeal_components:MX-Choc-1U" H 3050 4900 50  0001 C CNN
+F 2 "xeal_components:MX-Choc-1.5U" H 3050 4900 50  0001 C CNN
 F 3 "~" H 3050 4900 50  0001 C CNN
 	1    3050 4900
@@
 F 0 "K56" H 3550 5150 50  0000 C CNN
 F 1 "FN2" H 3550 5044 50  0000 C CNN
-F 2 "xeal_components:MX-Choc-1U" H 3550 4900 50  0001 C CNN
+F 2 "xeal_components:MX-Alps-Choc-2U-stabflip-pinflip" H 3550 4900 50  0001 C CNN
 F 3 "~" H 3550 4900 50  0001 C CNN
 	1    3550 4900
@@
 F 0 "K57" H 4050 5150 50  0000 C CNN
 F 1 "LSPC" H 4050 5044 50  0000 C CNN
-F 2 "xeal_components:MX-Alps-Choc-2U-no-led" H 4050 4900 50  0001 C CNN
+F 2 "xeal_components:MX-Alps-Choc-2U-stabflip-pinflip" H 4050 4900 50  0001 C CNN
 F 3 "~" H 4050 4900 50  0001 C CNN
 	1    4050 4900
@@
 F 0 "K58" H 4550 5150 50  0000 C CNN
 F 1 "RSPC" H 4550 5044 50  0000 C CNN
-F 2 "xeal_components:MX-Alps-Choc-2U-no-led" H 4550 4900 50  0001 C CNN
+F 2 "xeal_components:MX-Alps-Choc-2U-stabflip-pinflip" H 4550 4900 50  0001 C CNN
 F 3 "~" H 4550 4900 50  0001 C CNN
 	1    4550 4900

Commit message: new: Rework pcb, remove all traces as keys are now flipped
Parts:
- D1, D10, D11, D12, D13, D14, D15, D16, D17, D18, D19, D2, D20, D21, D22, D23, D24, D25, D26, D27, D28, D29, D3, D30, D31, D32, D33, D34, D35, D36, D37, D38, D39, D4, D40, D41, D42, D43, D44, D45, D46, D47, D48, D49, D5, D50, D51, D52, D53, D54, D55, D56, D57, D58, D59, D6, D60, D61, D62, D63, D64, D65, D7, D8, D9: footprint xeal_components:D_DO-34_SOD68_P10.16mm_Horizontal_NoK -> Keebio-Parts:Diode-dual
- K1, K10, K11, K12, K13, K15, K16, K17, K18, K19, K2, K20, K21, K22, K23, K24, K25, K26, K28, K29, K3, K30, K31, K32, K33, K34, K35, K36, K37, K38, K4, K41, K42, K43, K44, K45, K46, K47, K48, K49, K5, K50, K59, K6, K60, K64, K7, K8, K9: footprint xeal_components:MX-Choc-1U -> Keebio-Parts:Kailh-PG1350-1u-NoLED
- K14, K51, K52, K53, K54, K55: footprint xeal_components:MX-Choc-1.5U -> xeal_components:Kailh-PG1350-1.5u-NoLED
- K27: footprint xeal_components:MX-Alps-Choc-2U-pin-flip -> Keebio-Parts:Kailh-PG1350-2u-NoLED
- K39, K65: footprint xeal_components:MX-Alps-Choc-2U-no-led -> Keebio-Parts:Kailh-PG1350-2u-NoLED
- K40: footprint xeal_components:MX-Choc-2.5U-pin21 -> xeal_components:Kailh-PG1350-2.5u-NoLED
- K56, K57, K58: footprint xeal_components:MX-Alps-Choc-2U-stabflip-pinflip -> Keebio-Parts:Kailh-PG1350-2u-NoLED
- K61, K62, K63: footprint xeal_components:MX-Choc-1U-pin-flip -> Keebio-Parts:Kailh-PG1350-1u-NoLED
