File: matrix.sch (KiCad schematic (older format))
At the start: 130 parts, among them K1 ESC, K10 #9, K11 #0, K12 MINUS, K13 PLUS, K14 TAB, K15 Q, K16 W, K17 E, K18 R, K19 T, K2 #1, K20 Y, K21 U, K22 I, K23 O, K24 P, K25 [, K26 ], K27 CAPS, K28 A, K29 S, K3 #2, K30 D, K31 F, K32 G, K33 H, K34 J, K35 K, K36 L, K37 SEMICOLON, K38 QUOTE, K39 ENTER, K4 #3, K40 LSHIFT, K41 Z, K42 X, K43 C, K44 V, K45 B, K46 N, K47 M, K48 COMMA, K49 DOT, K5 #4, K50 SLASH, K51 RSHIFT, K52 BACKSLASH, K53 LCTL, K54 LGUI, K55 LALT, K56 FN2, K57 LSPC, K58 RSPC, K59 RALT, K6 #5, K60 RGUI, K61 LEFT, K62 DOWN, K63 RIGHT, K64 UP, K65 BKSPC, K7 #6, K8 #7, K9 #8

Commit message: Fully connected PCB
Parts:
- K1, K10, K11, K12, K13, K15, K16, K17, K18, K19, K2, K20, K21, K22, K23, K24, K25, K26, K28, K29, K3, K30, K31, K32, K33, K34, K35, K36, K37, K38, K4, K41, K42, K43, K44, K45, K46, K47, K48, K49, K5, K50, K59, K6, K60, K61, K62, K63, K64, K7, K8, K9: footprint Keebio-Parts:Kailh-PG1350-1u-NoLED -> xeal_components:Kailh-PG1350-1u-NoLED

Commit message: new: Add text
Parts:
- D1, D10, D11, D12, D13, D14, D15, D16, D17, D18, D19, D2, D20, D21, D22, D23, D24, D25, D26, D27, D28, D29, D3, D30, D31, D32, D33, D34, D35, D36, D37, D38, D39, D4, D40, D41, D42, D43, D44, D45, D46, D47, D48, D49, D5, D50, D51, D52, D53, D54, D55, D56, D57, D58, D59, D6, D60, D61, D62, D63, D64, D65, D7, D8, D9: footprint Keebio-Parts:Diode-dual -> xeal_components:Diode-dual
- K27, K39, K58, K65: footprint Keebio-Parts:Kailh-PG1350-2u-NoLED -> xeal_components:Kailh-PG1350-2u-NoLED
- K56: footprint Keebio-Parts:Kailh-PG1350-2u-NoLED -> xeal_components:Kailh-PG1350-1.5u-NoLED
- K57: footprint Keebio-Parts:Kailh-PG1350-2u-NoLED -> xeal_components:Kailh-PG1350-2.5u-NoLED
