File: mf68.kicad_pcb (KiCad board)
At the start: 2 copper layers, 308 x 95.2 mm, 133 parts, among them K1 ESC, K10 #9, K11 #0, K12 MINUS, K13 PLUS, K14 TAB, K15 Q, K16 W, K17 E, K18 R, K19 T, K2 #1, K20 Y, K21 U, K22 I, K23 O, K24 P, K25 [, K26 ], K27 CAPS, K28 A, K29 S, K3 #2, K30 D, K31 F, K32 G, K33 H, K34 J, K35 K, K36 L, K37 SEMICOLON, K38 QUOTE, K39 ENTER, K4 #3, K40 LSHIFT, K41 Z, K42 X, K43 C, K44 V, K45 B, K46 N, K47 M, K48 COMMA, K49 DOT, K5 #4, K50 SLASH, K51 RSHIFT, K52 BACKSLASH, K53 LCTL, K54 LGUI, K55 LALT, K56 FN2, K57 LSPC, K58 RSPC, K59 RALT, K6 #5, K60 RGUI, K61 LEFT, K62 DOWN, K63 RIGHT, K64 UP, K65 BKSPC, K7 #6, K8 #7, K9 #8, U1 nice_nano

Commit message: new: Add mounting points to pcb
Parts:
- moved D14 3.11 mm to (56.0, 92.7)
Routing:
- net Net-(D14-Pad2): track 15.8 -> 10.00 mm
- net row4: track 470.9 -> 466.9 mm
- net row1: track 329.2 -> 332.7 mm
- net col2: track 365.9 -> 364.5 mm
Other:
- board size 308 x 95.2 mm -> 315 x 106 mm

Commit message: Add border
Parts:
- moved POWER_SW1 0.82 mm to (329.0, 107.8)
- moved U1 0.08 mm to (329.0, 78.0)
Routing:
- net Net-(BT1-Pad2): track 12.5 -> 11.7 mm
- net Net-(POWER_SW1-Pad1): track 50.3 -> 50.9 mm
Other:
- outline, holes or cut-outs redrawn

Commit message: Use m2 mounting holes
Parts:
- added REF**: m2, xeal_components:MountingHole_2.2mm_M2, F.Cu at (341.0, 109.5)
- added REF**: m2, xeal_components:MountingHole_2.2mm_M2, F.Cu at (321.5, 57.5)
- added REF**: m2, xeal_components:MountingHole_2.2mm_M2, F.Cu at (300.5, 57.5)
- added REF**: m2, xeal_components:MountingHole_2.2mm_M2, F.Cu at (230.5, 57.5)
- added REF**: m2, xeal_components:MountingHole_2.2mm_M2, F.Cu at (160.5, 57.5)
- added REF**: m2, xeal_components:MountingHole_2.2mm_M2, F.Cu at (90.5, 57.5)
- added REF**: m2, xeal_components:MountingHole_2.2mm_M2, F.Cu at (30.5, 57.5)
- added REF**: m2, xeal_components:MountingHole_2.2mm_M2, F.Cu at (30.5, 108.0)
- added REF**: m2, xeal_components:MountingHole_2.2mm_M2, F.Cu at (230.5, 158.0)
- added REF**: m2, xeal_components:MountingHole_2.2mm_M2, F.Cu at (300.5, 158.0)
- added REF**: m2, xeal_components:MountingHole_2.2mm_M2, F.Cu at (30.5, 158.0)
- added REF**: m2, xeal_components:MountingHole_2.2mm_M2, F.Cu at (160.5, 158.0)
- added REF**: m2, xeal_components:MountingHole_2.2mm_M2, F.Cu at (90.5, 158.0)
- added REF**: m2, xeal_components:MountingHole_2.2mm_M2, F.Cu at (341.0, 158.0)
- added REF**: m2, xeal_components:MountingHole_2.2mm_M2, F.Cu at (337.0, 57.5)
Other:
- outline, holes or cut-outs redrawn

Commit message: new: Rework pcb, remove all traces as keys are now flipped
Parts:
- removed REF** (x15): m2, xeal_components:MountingHole_2.2mm_M2
- D1, D10, D11, D12, D13, D14, D15, D16, D17, D18, D19, D2, D20, D21, D22, D23, D24, D25, D26, D27, D28, D29, D3, D30, D31, D32, D33, D34, D35, D36, D37, D38, D39, D4, D40, D41, D42, D43, D44, D45, D46, D47, D48, D49, D5, D50, D51, D52, D53, D54, D55, D56, D57, D58, D59, D6, D60, D61, D62, D63, D64, D65, D7, D8, D9: footprint xeal_components:D_DO-34_SOD68_P10.16mm_Horizontal_NoK -> Keebio-Parts:Diode-dual
- K1, K10, K11, K12, K13, K15, K16, K17, K18, K19, K2, K20, K21, K22, K23, K24, K25, K26, K28, K29, K3, K30, K31, K32, K33, K34, K35, K36, K37, K38, K4, K41, K42, K43, K44, K45, K46, K47, K48, K49, K5, K50, K59, K6, K60, K64, K7, K8, K9: footprint xeal_components:MX-Choc-1U -> Keebio-Parts:Kailh-PG1350-1u-NoLED
- K14, K51, K52, K53, K54, K55: footprint xeal_components:MX-Choc-1.5U -> xeal_components:Kailh-PG1350-1.5u-NoLED
- K27: footprint xeal_components:MX-Alps-Choc-2U-pin-flip -> Keebio-Parts:Kailh-PG1350-2u-NoLED
- K39, K65: footprint xeal_components:MX-Alps-Choc-2U-no-led -> Keebio-Parts:Kailh-PG1350-2u-NoLED
- K40: footprint xeal_components:MX-Choc-2.5U-pin21 -> xeal_components:Kailh-PG1350-2.5u-NoLED
- K56, K57, K58: footprint xeal_components:MX-Alps-Choc-2U-stabflip-pinflip -> Keebio-Parts:Kailh-PG1350-2u-NoLED
- K61, K62, K63: footprint xeal_components:MX-Choc-1U-pin-flip -> Keebio-Parts:Kailh-PG1350-1u-NoLED
- moved D1 3.88 mm to (52.4, 69.8)
- moved D2 3.72 mm to (71.4, 69.8)
- moved K63 0.47 mm to (328.6, 146.1)
- moved K62 0.47 mm to (309.6, 146.1)
- moved K64 0.47 mm to (309.6, 127.0)
- moved K39 0.47 mm to (300.0, 108.0)
- moved K51 0.47 mm to (285.8, 127.0)
- moved K60 0.47 mm to (261.9, 146.1)
- moved K26 0.47 mm to (281.0, 88.9)
- moved K38 0.47 mm to (271.5, 108.0)
- moved K50 0.47 mm to (261.9, 127.0)
- moved K59 0.47 mm to (242.9, 146.1)
- moved K25 0.47 mm to (261.9, 88.9)
- moved K37 0.47 mm to (252.4, 108.0)
- moved K49 0.47 mm to (242.9, 127.0)
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Routing:
- net row4: track 466.9 -> 0.00 mm, vias 1 -> 0
- net col0: track 402.7 -> 0.00 mm
- net row3: track 386.1 -> 0.00 mm, vias 1 -> 0
- net col1: track 384.1 -> 0.00 mm
- net col2: track 364.5 -> 0.00 mm, vias 1 -> 0
- net col3: track 353.3 -> 0.00 mm, vias 1 -> 0
- net row2: track 349.8 -> 0.00 mm, vias 1 -> 0
- net col4: track 347.3 -> 0.00 mm, vias 1 -> 0
- net col7: track 343.7 -> 0.00 mm
- net col5: track 333.2 -> 0.00 mm, vias 1 -> 0
- net row1: track 332.7 -> 0.00 mm
- net col8: track 331.1 -> 0.00 mm
- net col6: track 322.1 -> 0.00 mm, vias 1 -> 0
- net col9: track 311.8 -> 0.00 mm
- net row0: track 304.9 -> 0.00 mm
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
Commit message: Fully connected PCB
Parts:
- K1, K10, K11, K12, K13, K15, K16, K17, K18, K19, K2, K20, K21, K22, K23, K24, K25, K26, K28, K29, K3, K30, K31, K32, K33, K34, K35, K36, K37, K38, K4, K41, K42, K43, K44, K45, K46, K47, K48, K49, K5, K50, K59, K6, K60, K61, K62, K63, K64, K7, K8, K9: footprint Keebio-Parts:Kailh-PG1350-1u-NoLED -> xeal_components:Kailh-PG1350-1u-NoLED
- moved D65 34.4 mm to (317.5, 69.8)
- moved D27 9.62 mm to (70.6, 107.9)
- moved D52 6.31 mm to (295.2, 88.8), turned to 90 degrees
- moved D53 6.23 mm to (61.9, 146.0)
- moved D55 6.19 mm to (119.1, 146.1)
- moved D54 6.19 mm to (90.5, 146.1)
- moved D56 4.61 mm to (156.4, 146.1)
- moved D58 4.32 mm to (232.6, 146.0)
- moved D57 4.17 mm to (194.5, 146.0)
- moved D3 4.04 mm to (90.5, 69.8)
- moved D38 4.04 mm to (281.0, 107.9)
- moved D39 4.04 mm to (283.4, 107.9)
- moved D59 4.00 mm to (252.4, 146.0)
- moved D62 4.00 mm to (300.0, 146.0)
- moved D63 4.00 mm to (319.1, 146.0)
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Connections:
- U1 pad 1: row1 -> col6
- U1 pad 13: col6 -> col4
- U1 pad 15: col4 -> row1
- U1 pad 16: col3 -> col0
- U1 pad 17: col2 -> col1
- U1 pad 18: col1 -> col2
- U1 pad 19: col0 -> col3
Routing:
- net row4: track 0.00 -> 422.2 mm
- net col0: track 0.00 -> 381.6 mm
- net col1: track 0.00 -> 368.2 mm
- net col6: track 0.00 -> 345.6 mm, vias 0 -> 1
- net col2: track 0.00 -> 344.1 mm
- net col3: track 0.00 -> 335.9 mm
- net row3: track 0.00 -> 334.2 mm, vias 0 -> 2
- net col7: track 0.00 -> 327.6 mm, vias 0 -> 1
- net col4: track 0.00 -> 324.0 mm
- net col5: track 0.00 -> 324.0 mm
- net col8: track 0.00 -> 312.2 mm, vias 0 -> 1
- net row2: track 0.00 -> 303.4 mm
- net row0: track 0.00 -> 297.5 mm
- net col9: track 0.00 -> 291.2 mm, vias 0 -> 1
- net row1: track 0.00 -> 285.9 mm
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
Commit message: new: Add text
Parts:
- D1, D10, D11, D12, D13, D14, D15, D16, D17, D18, D19, D2, D20, D21, D22, D23, D24, D25, D26, D27, D28, D29, D3, D30, D31, D32, D33, D34, D35, D36, D37, D38, D39, D4, D40, D41, D42, D43, D44, D45, D46, D47, D48, D49, D5, D50, D51, D52, D53, D54, D55, D56, D57, D58, D59, D6, D60, D61, D62, D63, D64, D65, D7, D8, D9: footprint Keebio-Parts:Diode-dual -> xeal_components:Diode-dual
- K27, K39, K58, K65: footprint Keebio-Parts:Kailh-PG1350-2u-NoLED -> xeal_components:Kailh-PG1350-2u-NoLED
- K56: footprint Keebio-Parts:Kailh-PG1350-2u-NoLED -> xeal_components:Kailh-PG1350-1.5u-NoLED
- K57: footprint Keebio-Parts:Kailh-PG1350-2u-NoLED -> xeal_components:Kailh-PG1350-2.5u-NoLED
- moved D56 8.73 mm to (147.6, 146.1)
- moved K57 4.76 mm to (171.4, 146.1)
- moved K56 4.74 mm to (133.3, 146.1)
Routing:
- net Net-(D57-Pad2): track 19.1 -> 25.1 mm
- net col3: track 335.9 -> 331.2 mm
- net row4: track 422.2 -> 418.1 mm
- net Net-(D56-Pad2): track 19.1 -> 15.1 mm
- net col4: track 324.0 -> 325.4 mm

Commit message: new: prepare for export to jlcpcb
Parts:
- added REF**: m2, xeal_components:MountingHole_2.2mm_M2, F.Cu at (322.0, 58.0)
- added REF**: m2, xeal_components:MountingHole_2.2mm_M2, F.Cu at (280.0, 158.0)
- added REF**: m2, xeal_components:MountingHole_2.2mm_M2, F.Cu at (156.0, 158.0)
- added REF**: m2, xeal_components:MountingHole_2.2mm_M2, F.Cu at (93.0, 158.0)
- added REF**: m2, xeal_components:MountingHole_2.2mm_M2, F.Cu at (31.0, 108.0)
- added REF**: m2, xeal_components:MountingHole_2.2mm_M2, F.Cu at (341.0, 158.0)
- added REF**: m2, xeal_components:MountingHole_2.2mm_M2, F.Cu at (31.0, 158.0)
- added REF**: m2, xeal_components:MountingHole_2.2mm_M2, F.Cu at (341.0, 108.0)
- added REF**: m2, xeal_components:MountingHole_2.2mm_M2, F.Cu at (337.0, 58.0)
- added REF**: m2, xeal_components:MountingHole_2.2mm_M2, F.Cu at (280.0, 58.0)
- added REF**: m2, xeal_components:MountingHole_2.2mm_M2, F.Cu at (218.0, 58.0)
- added REF**: m2, xeal_components:MountingHole_2.2mm_M2, F.Cu at (156.0, 58.0)
- added REF**: m2, xeal_components:MountingHole_2.2mm_M2, F.Cu at (31.0, 58.0)
- added REF**: m2, xeal_components:MountingHole_2.2mm_M2, F.Cu at (93.0, 58.0)
- added REF**: m2, xeal_components:MountingHole_2.2mm_M2, F.Cu at (218.0, 158.0)
Routing:
- net col12: track 169.0 -> 166.7 mm
- net row3: track 334.2 -> 335.7 mm
